Commit message: remove __pycache__

File: output/label42.urdf (robot description, URDF)
Before this commit: robot my_urdf, 22 links, 21 joints
Joints:
- joint knob11_to_drawer0: limit lower=0 upper=0.4 effort=5 velocity=2.283 -> lower=0 upper=1.57 effort=5 velocity=2.283
- joint knob12_to_drawer8: limit lower=0 upper=0.4 effort=5 velocity=2.283 -> lower=0 upper=1.57 effort=5 velocity=2.283
- joint knob13_to_drawer6: limit lower=0 upper=0.4 effort=5 velocity=2.283 -> lower=0 upper=1.57 effort=5 velocity=2.283
- joint knob15_to_drawer4: limit lower=0 upper=0.4 effort=5 velocity=2.283 -> lower=0 upper=1.57 effort=5 velocity=2.283
- joint knob16_to_drawer3: limit lower=0 upper=0.4 effort=5 velocity=2.283 -> lower=0 upper=1.57 effort=5 velocity=2.283
- joint knob17_to_doorR2: limit lower=0 upper=0.4 effort=5 velocity=2.283 -> lower=0 upper=1.57 effort=5 velocity=2.283
- joint knob18_to_drawer1: limit lower=0 upper=0.4 effort=5 velocity=2.283 -> lower=0 upper=1.57 effort=5 velocity=2.283
- joint knob19_to_drawer9: limit lower=0 upper=0.4 effort=5 velocity=2.283 -> lower=0 upper=1.57 effort=5 velocity=2.283
- joint knob20_to_drawer10: limit lower=0 upper=0.4 effort=5 velocity=2.283 -> lower=0 upper=1.57 effort=5 velocity=2.283
